Commit message: meshes and urdf files merged in one folder and scripts modified for relative paths

File: data/simulation_models/acromonk.urdf (robot description, URDF)
Before this commit: robot acromonk, 7 links, 7 joints
Links:
- link Base: geometry visual mesh filename=meshes/Base.obj
- link IMU: geometry visual mesh filename=meshes/IMU.obj
- link hook_1: geometry visual mesh filename=meshes/hook_1.obj
- link hook_2: geometry visual mesh filename=meshes/hook_2.obj
- link link_2: geometry visual mesh filename=meshes/link_2.obj
- link stick_1: geometry visual mesh filename=meshes/stick_1.obj
- link stick_2: geometry visual mesh filename=meshes/stick_2.obj
